File: PCB/heidi-pico/heidi-pico.kicad_sch (KiCad schematic)
At the start: 32 parts, among them J1 USB_C_Receptacle_USB2.0_14P, J2 Conn_01x03, J3 Conn_01x20, J4 Conn_01x20, SW1 SW_Push, U1 RP2040, U2 MCP1700x-330xxTT, U3 W25Q16JVZPIQ TR, Y1 ABM8-272-T3

Commit message: a
Parts:
- added D1: LED, LED_SMD:LED_0603_1608Metric, symbol Device:LED
- added R8: 91, Resistor_SMD:R_0603_1608Metric, symbol Device:R_Small
- added U4: DS18B20U, Package_SO:MSOP-8_3x3mm_P0.65mm, symbol Sensor_Temperature:DS18B20U
Connections:
- net +3V3: now also U4.8 (V_{DD})
- net GND: now also D1.2 (A), U4.4 (GND)
- net VBUS: now also R8.1
- net GPIO25: now reaches U1.37 (GPIO25)
- net GPIO25: now also U4.1 (DQ)
- new net: D1.1 (K), R8.2
- no-connect marks 1 -> 0
